Commit message: 添加闭链 mimic joint

File: Mos/urdf/mos_leg_51/urdf/mos_leg_51.urdf (robot description, URDF)
Before this commit: robot mos_leg_51, 8 links, 7 joints
Links:
- link front_gear: geometry collision mesh filename=../meshes/front_gear.STL; visual mesh filename=../meshes/front_gear.STL
- link hip_body: geometry collision mesh filename=../meshes/hip_body.STL; visual mesh filename=../meshes/hip_body.STL
- link hip_motor: geometry collision mesh filename=../meshes/hip_motor.STL; visual mesh filename=../meshes/hip_motor.STL
- link rear_gear: geometry collision mesh filename=../meshes/rear_gear.STL; visual mesh filename=../meshes/rear_gear.STL
- link shank: geometry collision mesh filename=../meshes/shank.STL; visual mesh filename=../meshes/shank.STL
- link shank_gear: geometry collision mesh filename=../meshes/shank_gear.STL; visual mesh filename=../meshes/shank_gear.STL
- link shank_link: geometry collision mesh filename=../meshes/shank_link.STL; visual mesh filename=../meshes/shank_link.STL
- link thigh: geometry collision mesh filename=../meshes/thigh.STL; visual mesh filename=../meshes/thigh.STL
